Commit message: Xarco Fixes.

File: src/crustcrawler_description/urdf/crustcrawler.xacro (robot description, xacro)
@@ -189,11 +189,11 @@
   <link name="gripper_left">
     <collision>
-      <origin xyz="0 0 1" rpy="0 0 0"/>
-      <geometry>
-        <box size=" ${LinkWidth} ${LinkWidth} ${LinkWidth}"/>
-      </geometry>
-    </collision>
-    <visual>
-      <origin xyz="${-L3 + 0.001} 0.016   0" rpy="${M_pi/2} 0 ${M_pi/2}"/>
+      <origin xyz="0 0 0" rpy="0 0 0"/>
+      <geometry>
+        <mesh filename="package://crustcrawler_description/meshes/Grip.STL"/>
+      </geometry>
+    </collision>
+    <visual>
+      <origin xyz="0 0 0" rpy="0 0 0"/>
       <geometry>
         <mesh filename="package://crustcrawler_description/meshes/Grip.STL"/>
@@ -212,11 +212,11 @@
   <link name="gripper_right">
     <collision>
-      <origin xyz="0 0 1" rpy="0 0 0"/>
-      <geometry>
-        <box size=" ${LinkWidth} ${LinkWidth} ${LinkWidth}"/>
-      </geometry>
-    </collision>
-    <visual>
-      <origin xyz="${-L3 + 0.001} -0.016  0" rpy="${-M_pi/2} 0 ${-M_pi/2}"/>
+      <origin xyz="0 0 0" rpy="${M_pi} 0 0"/>
+      <geometry>
+        <mesh filename="package://crustcrawler_description/meshes/Grip.STL"/>
+      </geometry>
+    </collision>
+    <visual>
+      <origin xyz="0 0 0" rpy="${M_pi} 0 0"/>
       <geometry>
         <mesh filename="package://crustcrawler_description/meshes/Grip.STL"/>

Commit message: put in dynamics

File: src/crustcrawler_description/urdf/crustcrawler.xacro (robot description, xacro)
@@ -69,5 +69,5 @@
     </inertial>
   </link>
-  <joint name="joint1" type="continuous">
+  <joint name="joinposRobot[0]" type="continuous">
     <axis xyz="0 0 1"/>
     <!--limit effort="1000.0" lower="${-M_pi}" upper="${M_pi}" velocity="0.5"/ -->

Commit message: URDF file should work now, but who knows.

File: src/crustcrawler_description/urdf/crustcrawler.xacro (robot description, xacro)
@@ -39,4 +39,10 @@
     <selfCollide>true</selfCollide>
   </gazebo>
+  <gazebo reference="gripper_left">
+    <selfCollide>true</selfCollide>
+  </gazebo>
+  <gazebo reference="gripper_right">
+    <selfCollide>true</selfCollide>
+  </gazebo>
   <!-- links, joints and transmissions -->
   <link name="world"/>
@@ -148,5 +154,5 @@
       <origin xyz="${L3/2} 0 ${d3}" rpy="0 0 0"/>
       <geometry>
-        <box size=" ${L3 - MotorOffset*2} ${LinkWidth} ${LinkHeight}"/>
+        <box size=" ${L3 - MotorOffset*2} ${LinkWidth/2} ${LinkHeight}"/>
       </geometry>
     </collision>
@@ -154,5 +160,5 @@
       <origin xyz="${L3 - 0.01} 0 ${d3}" rpy="0 0 0"/>
       <geometry>
-        <box size=" ${0.045} ${MotorLength} ${MotorWidth*2 - 0.005}"/>
+        <box size=" ${0.045} ${MotorLength/2} ${MotorWidth*2 - 0.005}"/>
       </geometry>
     </collision>
@@ -183,5 +189,5 @@
     <parent link="link3"/>
     <child link="gripper_right"/>
-    <origin xyz="${L3 - 0.003} 0 -0.016" rpy="${-M_pi/2} 0 0"/>
+    <origin xyz="${L3 - 0.003} 0.003 -0.023" rpy="${-M_pi/2} 0 0"/>
     <dynamics damping="0.7"/>
   </joint> -->
@@ -212,5 +218,5 @@
   <link name="gripper_right">
     <collision>
-      <origin xyz="0 0 0" rpy="${M_pi} 0 0"/>
+      <origin xyz="0 0.0 0" rpy="${M_pi} 0 0"/>
       <geometry>
         <mesh filename="package://crustcrawler_description/meshes/Grip.STL"/>

Commit message: xacro fix

File: src/crustcrawler_description/urdf/crustcrawler.xacro (robot description, xacro)
@@ -75,5 +75,5 @@
     </inertial>
   </link>
-  <joint name="joinposRobot[0]" type="continuous">
+  <joint name="joint1" type="continuous">
     <axis xyz="0 0 1"/>
     <!--limit effort="1000.0" lower="${-M_pi}" upper="${M_pi}" velocity="0.5"/ -->

Commit message: add friction

File: src/crustcrawler_description/urdf/crustcrawler.xacro (robot description, xacro)
@@ -81,5 +81,5 @@
     <child link="link1"/>
     <origin xyz="0 0 0" rpy= "0 0 0"/>
-    <dynamics damping="0.7"/>
+    <dynamics damping="0.7" friction="50"/>
   </joint>
   <!-- link 1 -->
@@ -111,5 +111,5 @@
     <parent link="link1"/>
     <child link="link2"/>
-    <dynamics damping="0.7"/>
+    <dynamics damping="0.7" friction="50"/>
   </joint>
   <!-- link 2 -->
@@ -147,5 +147,5 @@
     <child link="link3"/>
     <origin xyz="${L2} 0 0" rpy="0 0 0"/>
-    <dynamics damping="0.7"/>
+    <dynamics damping="0.7" friction="50"/>
   </joint>
   <!-- link 3 -->

Commit message: fixed friction

File: src/crustcrawler_description/urdf/crustcrawler.xacro (robot description, xacro)
@@ -81,5 +81,5 @@
     <child link="link1"/>
     <origin xyz="0 0 0" rpy= "0 0 0"/>
-    <dynamics damping="0.7" friction="50"/>
+    <dynamics damping="0.7" friction="0.1"/>
   </joint>
   <!-- link 1 -->
@@ -111,5 +111,5 @@
     <parent link="link1"/>
     <child link="link2"/>
-    <dynamics damping="0.7" friction="50"/>
+    <dynamics damping="0.7" friction="0.1"/>
   </joint>
   <!-- link 2 -->
@@ -147,5 +147,5 @@
     <child link="link3"/>
     <origin xyz="${L2} 0 0" rpy="0 0 0"/>
-    <dynamics damping="0.7" friction="50"/>
+    <dynamics damping="0.7" friction="0.1"/>
   </joint>
   <!-- link 3 -->
@@ -183,5 +183,5 @@
     <child link="gripper_left"/>
     <origin xyz="${L3 - 0.003} 0 0.016" rpy="${-M_pi/2} 0 0"/>
-    <dynamics damping="0.7"/>
+    <dynamics damping="0.7" friction="0.1"/>
   </joint>
   <joint name="joint5" type="continuous">
@@ -190,5 +190,5 @@
     <child link="gripper_right"/>
     <origin xyz="${L3 - 0.003} 0.003 -0.023" rpy="${-M_pi/2} 0 0"/>
-    <dynamics damping="0.7"/>
+    <dynamics damping="0.7" friction="0.1"/>
   </joint> -->
   <!-- left gripper -->

Commit message: Updated masses and center of gravity

File: src/crustcrawler_description/urdf/crustcrawler.xacro (robot description, xacro)
@@ -14,11 +14,11 @@
   <xacro:property name="L3" value="0.15" />
   <xacro:property name="Lp" value="0.0" />
-  <xacro:property name="Lc" value="0.05875" />
+  <xacro:property name="Lc" value="0.02895" />
   <xacro:property name="Lc2" value="0.17433" />
   <xacro:property name="Lc3" value="0.12078" />
   <xacro:property name="d3" value="-0.003" />
-  <xacro:property name="m1" value="0.22501148645" />
-  <xacro:property name="m2" value="0.21285774246" />
-  <xacro:property name="m3" value="0.28725035108" />
+  <xacro:property name="m1" value="0.1874" />
+  <xacro:property name="m2" value="0.17226" />
+  <xacro:property name="m3" value="0.18391" />
   <xacro:property name="mp" value="0.0" />
   <!-- Gazebo -->

Commit message: changed frames and visual stuff

File: src/crustcrawler_description/urdf/crustcrawler.xacro (robot description, xacro)
@@ -107,5 +107,5 @@
   </link>
   <joint name="joint2" type="continuous">
-    <origin xyz="0 0 ${L1}" rpy="${M_pi / 2} 0 0"/>
+    <origin xyz="0 0 ${L1}" rpy="${-M_pi / 2} 0 0"/>
     <axis xyz="0 0 1"/>
     <parent link="link1"/>
@@ -128,5 +128,5 @@
     </collision>
     <visual>
-      <origin xyz="0 0 0.002" rpy="0 ${M_pi/2} 0"/>
+      <origin xyz="0 0 -0.002" rpy="${M_pi/2} ${-M_pi/2} ${M_pi/2}"/>
       <geometry>
 	       <mesh filename="package://crustcrawler_description/meshes/Link2.STL"/> <!--<box size="${L2} ${LinkWidth} ${LinkWidth}"/>-->
@@ -164,5 +164,5 @@
     </collision>
     <visual>
-      <origin xyz="0 0 0" rpy="0 ${M_pi/2} 0"/>
+      <origin xyz="0 0 0" rpy="${M_pi/2} ${-M_pi/2} ${M_pi/2}"/>
       <geometry>
         <mesh filename="package://crustcrawler_description/meshes/Link3.STL"/>
@@ -182,5 +182,5 @@
     <parent link="link3"/>
     <child link="gripper_left"/>
-    <origin xyz="${L3 - 0.003} 0 0.016" rpy="${-M_pi/2} 0 0"/>
+    <origin xyz="${L3 - 0.003} 0 0.016" rpy="${M_pi/2} 0 0"/>
     <dynamics damping="0.7" friction="0.1"/>
   </joint>
@@ -189,5 +189,5 @@
     <parent link="link3"/>
     <child link="gripper_right"/>
-    <origin xyz="${L3 - 0.003} 0.003 -0.023" rpy="${-M_pi/2} 0 0"/>
+    <origin xyz="${L3 - 0.003} 0.003 -0.023" rpy="${M_pi/2} 0 0"/>
     <dynamics damping="0.7" friction="0.1"/>
   </joint> -->
@@ -195,11 +195,11 @@
   <link name="gripper_left">
     <collision>
-      <origin xyz="0 0 0" rpy="0 0 0"/>
-      <geometry>
-        <mesh filename="package://crustcrawler_description/meshes/Grip.STL"/>
-      </geometry>
-    </collision>
-    <visual>
-      <origin xyz="0 0 0" rpy="0 0 0"/>
+      <origin xyz="0 0 0" rpy="${M_pi} 0 0"/>
+      <geometry>
+        <mesh filename="package://crustcrawler_description/meshes/Grip.STL"/>
+      </geometry>
+    </collision>
+    <visual>
+      <origin xyz="0 0 0" rpy="${M_pi} 0 0"/>
       <geometry>
         <mesh filename="package://crustcrawler_description/meshes/Grip.STL"/>
@@ -218,11 +218,11 @@
   <link name="gripper_right">
     <collision>
-      <origin xyz="0 0.0 0" rpy="${M_pi} 0 0"/>
-      <geometry>
-        <mesh filename="package://crustcrawler_description/meshes/Grip.STL"/>
-      </geometry>
-    </collision>
-    <visual>
-      <origin xyz="0 0 0" rpy="${M_pi} 0 0"/>
+      <origin xyz="0 0.0 0" rpy="0 0 0"/>
+      <geometry>
+        <mesh filename="package://crustcrawler_description/meshes/Grip.STL"/>
+      </geometry>
+    </collision>
+    <visual>
+      <origin xyz="0 0 0" rpy="0 0 0"/>
       <geometry>
         <mesh filename="package://crustcrawler_description/meshes/Grip.STL"/>

Commit message: fixed gravity compensation

File: src/crustcrawler_description/urdf/crustcrawler.xacro (robot description, xacro)
@@ -40,8 +40,8 @@
   </gazebo>
   <gazebo reference="gripper_left">
-    <selfCollide>true</selfCollide>
+    <selfCollide>false</selfCollide>
   </gazebo>
   <gazebo reference="gripper_right">
-    <selfCollide>true</selfCollide>
+    <selfCollide>false</selfCollide>
   </gazebo>
   <!-- links, joints and transmissions -->
@@ -107,5 +107,5 @@
   </link>
   <joint name="joint2" type="continuous">
-    <origin xyz="0 0 ${L1}" rpy="${-M_pi / 2} 0 0"/>
+    <origin xyz="0 0 ${L1}" rpy="${-M_pi / 2} ${-M_pi/2} ${M_pi}"/>
     <axis xyz="0 0 1"/>
     <parent link="link1"/>

Commit message: Inertia and masse of the grippers.

File: src/crustcrawler_description/urdf/crustcrawler.xacro (robot description, xacro)
@@ -208,9 +208,9 @@
     <inertial>
       <origin xyz="0 0 0 " rpy="0 0 0"/>
-      <mass value="0.001"/>
-      <inertia
-    ixx="0.0" ixy="0.0" ixz="0.0"
-    iyy="0.0" iyz="0.0"
-    izz="0.0"/>
+      <mass value="0.02965"/>
+      <inertia
+    ixx="7.98622000000000e-5" ixy="6.37430000000000e-6" ixz="-3.25600000000000e-7"
+                              iyy="0.000489436900000000" iyz=" 1.41040000000000e-6"
+                                                        izz="0.000461895400000000"/>
     </inertial>
   </link>
@@ -231,9 +231,9 @@
     <inertial>
       <origin xyz="0 0 0 " rpy="0 0 0"/>
-      <mass value="0.001"/>
-      <inertia
-    ixx="0.0" ixy="0.0" ixz="0.0"
-    iyy="0.0" iyz="0.0"
-    izz="0.0"/>
+      <mass value="0.02965"/>
+      <inertia
+    ixx="7.98622000000000e-5" ixy="6.37430000000000e-6" ixz="-3.25600000000000e-7"
+                              iyy="0.000489436900000000" iyz=" 1.41040000000000e-6"
+                                                        izz="0.000461895400000000"/>
     </inertial>
   </link>

Commit message: joint fix

File: src/crustcrawler_description/urdf/crustcrawler.xacro (robot description, xacro)
@@ -81,12 +81,12 @@
     <child link="link1"/>
     <origin xyz="0 0 0" rpy= "0 0 0"/>
-    <dynamics damping="0.7" friction="0.1"/>
+    <dynamics damping="0.7" friction="0.0"/>
   </joint>
   <!-- link 1 -->
   <link name="link1">
     <collision>
-      <origin xyz="0 0 ${L1 / 2}" rpy="0 0 0"/>
-      <geometry>
-        <box size="${MotorWidth} ${MotorLength} ${L1*1.5}"/>
+      <origin xyz="0 0 ${L1 / 1.8}" rpy="0 0 0"/>
+      <geometry>
+        <box size="${MotorWidth} ${MotorLength} ${L1*1.3}"/>
       </geometry>
     </collision>
@@ -182,5 +182,5 @@
     <parent link="link3"/>
     <child link="gripper_left"/>
-    <origin xyz="${L3 - 0.003} 0 0.016" rpy="${M_pi/2} 0 0"/>
+    <origin xyz="${L3 - 0.003} -0.0015 0.022" rpy="${M_pi/2} 0 0"/>
     <dynamics damping="0.7" friction="0.1"/>
   </joint>
@@ -189,5 +189,5 @@
     <parent link="link3"/>
     <child link="gripper_right"/>
-    <origin xyz="${L3 - 0.003} 0.003 -0.023" rpy="${M_pi/2} 0 0"/>
+    <origin xyz="${L3 - 0.003} 0.0015 -0.0165" rpy="${M_pi/2} 0 0"/>
     <dynamics damping="0.7" friction="0.1"/>
   </joint> -->
@@ -233,7 +233,7 @@
       <mass value="0.001"/>
       <inertia
-    ixx="0.0" ixy="0.0" ixz="0.0"
-    iyy="0.0" iyz="0.0"
-    izz="0.0"/>
+    ixx="0.00000001" ixy="0.00000001" ixz="0.00000001"
+    iyy="0.00000001" iyz="0.00000001"
+    izz="0.00000001"/>
     </inertial>
   </link>

Commit message: inertia fix

File: src/crustcrawler_description/urdf/crustcrawler.xacro (robot description, xacro)
@@ -210,7 +210,7 @@
       <mass value="0.02965"/>
       <inertia
-    ixx="7.98622000000000e-5" ixy="6.37430000000000e-6" ixz="-3.25600000000000e-7"
-                              iyy="0.000489436900000000" iyz=" 1.41040000000000e-6"
-                                                        izz="0.000461895400000000"/>
+        ixx="0.0000798622" ixy="0.0000063743" ixz="-0.0000003256"
+                   iyy="0.000489436900000000" iyz=" 0.0000014104"
+                                       izz="0.000461895400000000"/>
     </inertial>
   </link>
@@ -233,14 +233,8 @@
       <mass value="0.02965"/>
       <inertia
-<<<<<<< HEAD
-    ixx="0.00000001" ixy="0.00000001" ixz="0.00000001"
-    iyy="0.00000001" iyz="0.00000001"
-    izz="0.00000001"/>
-=======
-    ixx="7.98622000000000e-5" ixy="6.37430000000000e-6" ixz="-3.25600000000000e-7"
-                              iyy="0.000489436900000000" iyz=" 1.41040000000000e-6"
-                                                        izz="0.000461895400000000"/>
->>>>>>> 925c992d149f682f64b2c523561ff3dc2555c0f5
-    </inertial>
+        ixx="0.0000798622" ixy="0.0000063743" ixz="-0.0000003256"
+                 iyy="0.000489436900000000" iyz=" 0.0000014104"
+                                     izz="0.000461895400000000" />
+     </inertial>
   </link>
 </robot>

Commit message: Control Fixes.

File: src/crustcrawler_description/urdf/crustcrawler.xacro (robot description, xacro)
@@ -81,5 +81,5 @@
     <child link="link1"/>
     <origin xyz="0 0 0" rpy= "0 0 0"/>
-    <dynamics damping="0.7" friction="0.0"/>
+    <dynamics damping="0.7" friction="0.1"/>
   </joint>
   <!-- link 1 -->

Commit message: Better daminping and frictions values for gazebo.

File: src/crustcrawler_description/urdf/crustcrawler.xacro (robot description, xacro)
@@ -81,5 +81,5 @@
     <child link="link1"/>
     <origin xyz="0 0 0" rpy= "0 0 0"/>
-    <dynamics damping="0.7" friction="0.1"/>
+    <dynamics damping="1.0" friction="0.4"/>
   </joint>
   <!-- link 1 -->
@@ -111,5 +111,5 @@
     <parent link="link1"/>
     <child link="link2"/>
-    <dynamics damping="0.7" friction="0.1"/>
+    <dynamics damping="1.0" friction="0.4"/>
   </joint>
   <!-- link 2 -->

Commit message: Simulation Fixes.

File: src/crustcrawler_description/urdf/crustcrawler.xacro (robot description, xacro)
@@ -182,5 +182,5 @@
     <parent link="link3"/>
     <child link="gripper_left"/>
-    <origin xyz="${L3 - 0.003} -0.0015 0.022" rpy="${M_pi/2} 0 0"/>
+    <origin xyz="${L3 - 0.003} -0.0015 0.022" rpy="${-M_pi/2} 0 0"/>
     <dynamics damping="0.7" friction="0.1"/>
   </joint>
@@ -189,5 +189,5 @@
     <parent link="link3"/>
     <child link="gripper_right"/>
-    <origin xyz="${L3 - 0.003} 0.0015 -0.0165" rpy="${M_pi/2} 0 0"/>
+    <origin xyz="${L3 - 0.003} 0.0015 -0.0165" rpy="${-M_pi/2} 0 0"/>
     <dynamics damping="0.7" friction="0.1"/>
   </joint> -->
@@ -195,11 +195,11 @@
   <link name="gripper_left">
     <collision>
-      <origin xyz="0 0 0" rpy="${M_pi} 0 0"/>
-      <geometry>
-        <mesh filename="package://crustcrawler_description/meshes/Grip.STL"/>
-      </geometry>
-    </collision>
-    <visual>
-      <origin xyz="0 0 0" rpy="${M_pi} 0 0"/>
+      <origin xyz="0 0 0" rpy="0 0 0"/>
+      <geometry>
+        <mesh filename="package://crustcrawler_description/meshes/Grip.STL"/>
+      </geometry>
+    </collision>
+    <visual>
+      <origin xyz="0 0 0" rpy="0 0 0"/>
       <geometry>
         <mesh filename="package://crustcrawler_description/meshes/Grip.STL"/>
@@ -218,11 +218,11 @@
   <link name="gripper_right">
     <collision>
-      <origin xyz="0 0.0 0" rpy="0 0 0"/>
-      <geometry>
-        <mesh filename="package://crustcrawler_description/meshes/Grip.STL"/>
-      </geometry>
-    </collision>
-    <visual>
-      <origin xyz="0 0 0" rpy="0 0 0"/>
+      <origin xyz="0 0.0 0" rpy="${M_pi} 0 0"/>
+      <geometry>
+        <mesh filename="package://crustcrawler_description/meshes/Grip.STL"/>
+      </geometry>
+    </collision>
+    <visual>
+      <origin xyz="0 0 0" rpy="${M_pi} 0 0"/>
       <geometry>
         <mesh filename="package://crustcrawler_description/meshes/Grip.STL"/>
